File: circuit/circuit.sch (KiCad schematic (older format))
At the start: 19 parts, among them J1 Connector to Heater, J2 RX/TX Connector, Q1 2N2219, Q2 IRF4905, SW1 Reset, SW2 Bootloader, U1 HT7833, U2 74HC74, U3 ESP-12E

Commit message: Arduino/C++ Code, FHEM Code and Pictures
Parts:
- removed D2: 9.1V, symbol D_Zener
- removed J2: RX/TX Connector, symbol Conn_01x04_Female
- removed Q1: 2N2219, TO_SOT_Packages_THT:TO-39-3, symbol 2N2219
- removed Q2: IRF4905, TO_SOT_Packages_THT:TO-220_Vertical, symbol IRF4905
- removed R1, R2: 100k, symbol R
- removed R3: 500, symbol R
- removed R4: 100, symbol R
- removed R5: 10k, symbol R
- removed SW1: Reset, symbol SW_DIP_x01
- removed SW2: Bootloader, symbol SW_DIP_x01
- removed U2: 74HC74, symbol 74HC74
- removed U3: ESP-12E, symbol ESP-12E
- added Q?: Q_PNP_BCE, symbol Q_PNP_BCE
- added Q?: Q_NPN_BCE, symbol Q_NPN_BCE
- added R?: 100k, symbol R
- added R?: 2,2k, symbol R
- added R?: 1k, symbol R
- added R?: 3k, symbol R
- added R?: 15k, symbol R
- added U?: ESP-12F, symbol ESP-12F
Connections:
- net +24V: now also D1.2 (A), J1.1 (Pin_1), Q?.3 (E), R?.1; no longer C1.1, D1.1 (K), U1.3 (VI)
- net Data: now also Q?.2 (C), R?.1
- net GND: now also Q?.3 (E), R?.1, U?.9 (GND)
- net VCC: now also C1.1, D1.1 (K), U1.3 (VI); no longer D1.2 (A), J1.1 (Pin_1)
- net +3V3 renamed +5V
- net +5V: now also U?.8 (VCC)
- new net: Q?.1 (B), R?.1, R?.2
- new net: Q?.1 (B), R?.1
- new net: Q?.2 (C), R?.2
- new net: R?.2, U?.12 (GPIO0)
- new net: R?.2, R?.2, U?.14 (GPIO5)
